File: peregrine.sch (EAGLE design)
At the start: 70 parts, among them IC2 LMV358IDGKR, J1 USB MICRO, U1 ITG-3200, U2 ADXL345, U4 3.3V, U5 ATMEGA32U4-XUAU, Y1 16MHz KX-7

Commit message: Many changes.
Added level conversion to schematic. Had to re-do route because of many
added components. Also, connected a number of things which needed
connections in schematic. Route about 80% done.
Parts:
- removed C25: 100n, SmartPrj:C-EUC0603
- removed JP3: (no value), pinhead:PINHD-2X2
- removed LED1: Blue, SparkFun:LED0603
- removed R3: 330, SparkFun:RESISTOR0402-RES
- removed RN1: 10K, resistor-dil:4R-NCAY16
- removed SJ1, SJ2, SJ3, SJ4: (no value), jumper:SJ
- removed U4: 3.3V, SparkFun:V_REG_LDOSMD
- added IC1: (no value), linear-technology:LT1129CST5
- added Q1, Q10, Q11, Q2: BSS123, transistor-small-signal:BSS123
- added R10, R4, R66, R67, R68, R69, R8, R9: 10k, SparkFun:RESISTOR0603-RES
- added R11, R12: 10k, resistor:R-US_R0603
- added SJ7, SJ8: (no value), SparkFun:SOLDERJUMPER_2WAYS
Connections:
- removed net 3.3V: C13.1, C14.1, U$3.VDDA, U$3.VDDD, U$4.VDDA, U$4.VDDD
- removed net A0: U5.(ADC7/TDI)PF7
- removed net A1: U5.(ADC6/TDO)PF6
- removed net A2: U5.(ADC5/TMS)PF5
- removed net A3: U5.(ADC4/TCK)PF4
- removed net A4: U5.(ADC1)PF1
- removed net A5: U5.(ADC0)PF0
- removed net D5*: U5.(OC3A/#0C4A)PC6
- removed net D6*: U5.(T0/OC4D/ADC10)PD7
- removed net GPS-RX: GPS.TX, SJ2.1
- removed net GPS-TX: GPS.RX, SJ1.1
- removed net IO10*: U5.(PCINT6/OC1B/OC4B/ADC13)PB6
- removed net IO12: U5.(T1/#OC4D/ADC9)PD6
- removed net IO8: U5.(ADC11/PCINT4)PB4
- removed net IO9*: U5.(PCINT5/OC1A/#OC4B/ADC12)PB5
- removed net M_1: JP1.2
- removed net M_2: JP2.2
- removed net M_3: JP4.2
- removed net M_4: JP1.1
- removed net M_AUX1: JP4.1
- removed net M_AUX2: JP2.1
- removed net N$10: U$3.SDA
- removed net N$13: U$3.SCL
- removed net N$15: U$4.SDA
- removed net N$16: U$4.SCL
- removed net N$4: LED1.C, R3.2
- removed net SCL: JP3.3, R2.1, SJ6.2, U$2.SCL, U1.SCL, U2.SCL, U5.(OC0B/SCL/INT0)PD0
- removed net SDA: JP3.1, R1.1, SJ5.2, U$2.SDA, U1.SDA, U2.SDA, U5.(SDA/INT1)PD1
- removed net VUSB: C27.+, C28.2, F1.1, U5.VBUS
- new net AT_RX3V3: Q1.S, R4.1, SJ8.3
- new net AT_TX3V3: Q2.S, R8.1, SJ7.3
- new net GPIO18(PCM_CLK): JP5.12
- new net GPS-INPUT: GPS.RX, SJ8.1
- new net GPS-OUTPUT: GPS.TX, SJ7.1
- new net MOT/SENS_1: JP1.1, U5.(ADC7/TDI)PF7
- new net MOT/SENS_2: JP1.2, U5.(ADC6/TDO)PF6
- new net MOT/SENS_3: JP2.1, U5.(ADC5/TMS)PF5
- new net MOT/SENS_4: JP2.2, U5.(ADC4/TCK)PF4
- new net MOT/SENS_5: JP4.1, U5.(ADC1)PF1
- new net MOT/SENS_6: JP4.2, U5.(ADC0)PF0
- new net SCL3V3: Q10.S, R2.1, R66.1, SJ6.2, U$2.SCL, U$3.SCL, U$4.SCL, U1.SCL, U2.SCL
- new net SCL5V: Q10.D, R69.1, U5.(OC0B/SCL/INT0)PD0
- new net SDA3V3: Q11.S, R1.1, R67.1, SJ5.2, U$2.SDA, U$3.SDA, U$4.SDA, U1.SDA, U2.SDA
- new net SDA5V: Q11.D, R68.1, U5.(SDA/INT1)PD1
- net +5V: now also C27.+, C28.2, F1.1, IC1G$1.IN, R10.2, R12.2, R68.2, R69.2, R9.2, U5.VBUS; no longer C25.1, JP3.2, RN1D.2, U4.EN, U4.IN
- net 3V3: now also C13.1, C14.1, IC1G$1.OUT, Q1.G, Q10.G, Q11.G, Q2.G, R4.2, R66.2, R67.2, R8.2, U$3.VDDA, U$3.VDDD, U$4.VDDA, U$4.VDDD; no longer LED1.A, U4.OUT
- net D0/RX: now also Q1.D, R10.1; no longer SJ2.2, SJ3.2
- net D1/TX: now also Q2.D, R9.1; no longer SJ1.2, SJ4.2
- net GND: now also IC1G$1.GND, R11.2; no longer C25.2, JP3.4, R3.1, RN1C.1, U4.GND
- net GPIO14(TXD): now also JP5.8, SJ8.2; no longer SJ3.1
- net GPIO15(RXD): now also JP5.10, SJ7.2; no longer SJ4.1
- net HWB: now also R11.1; no longer RN1C.2
- net REC1: now also U5.(T1/#OC4D/ADC9)PD6
- net REC2: now also U5.(T0/OC4D/ADC10)PD7
- net REC3: now also U5.(ADC11/PCINT4)PB4
- net REC4: now also U5.(PCINT5/OC1A/#OC4B/ADC12)PB5
- net REC5: now also U5.(PCINT6/OC1B/OC4B/ADC13)PB6
- net REC6: now also U5.(OC3A/#0C4A)PC6
- net RESET: now also R12.1; no longer RN1D.1
Other:
- moved on the sheet: C10, C11, C12, C27, C28, IC2A, L, ON, R1, R2, RN2A, RN2B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

Commit message: Fixed some stuff
Connections:
- new net GPIO23: JP5.16
- new net GPIO24: JP5.18
- new net GPIO25: JP5.22
- new net GPIO7(CE1): JP5.26
- new net GPIO8(CE0): JP5.24
- new net PI_5V: JP5.2
- new net PI_5V_2: JP5.4
- new net PI_GND3: JP5.6
- new net PI_GND4: JP5.14
- new net PI_GND5: JP5.20
